File: KiCAD/Seitenkonsole.kicad_sch (KiCad schematic)
At the start: 23 parts, among them SW1 Button, SW10 Button, SW11 Button, SW12 Button, SW13 Button, SW14 Button, SW15 Button, SW16 Button, SW17 Button, SW18 Button, SW19 Button, SW2 Button, SW20 Joystick, SW21 Joystick, SW22 Joystick_Switch, SW3 Button, SW4 Button, SW5 Button, SW6 Button, SW7 Button, SW8 Button, SW9 Button

Commit message: -
Connections:
- net D2: now also SW10.1, SW11.1, SW12.1, SW9.1; no longer SW1.1, SW2.1, SW3.1, SW4.1
- net D3: now also SW5.1, SW6.1, SW7.1, SW8.1; no longer SW13.1, SW14.1, SW15.1, SW16.1
- net D4: now also SW1.1, SW2.1, SW3.1, SW4.1; no longer SW17.1, SW18.1, SW19.1, SW22.S2
- net D5: now also SW13.1, SW14.1, SW15.1, SW16.1; no longer SW1.2, SW13.2, SW22.S1, SW5.2, SW9.2
- net D6: now also SW17.1, SW18.1, SW19.1, SW22.S2; no longer SW10.2, SW14.2, SW17.2, SW2.2, SW6.2
- net D7: now also SW1.2, SW13.2, SW22.S1, SW5.2, SW9.2; no longer SW11.2, SW15.2, SW18.2, SW3.2, SW7.2
- net D8: now also SW10.2, SW14.2, SW17.2, SW2.2, SW6.2; no longer SW12.2, SW16.2, SW19.2, SW4.2, SW8.2
- net D9: now reaches A1.24 (D9)
- net D9: now also SW11.2, SW15.2, SW18.2, SW3.2, SW7.2
- net D10: now reaches A1.25 (D10)
- net D10: now also SW12.2, SW16.2, SW19.2, SW4.2, SW8.2
- removed net D0: A1.15 (D0/RX), SW10.1, SW11.1, SW12.1, SW9.1
- removed net D1: A1.16 (D1/TX), SW5.1, SW6.1, SW7.1, SW8.1
- no-connect marks 15 -> 13

Commit message: -
Other:
- note added: "Col D7-D10 Row D2-D5"
- note added: "Joystick A0-A2"
Changed lines of the file:
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@@
     (stroke (width 0) (type default))
+  )
+  (text "Col D7-D10 Row D2-D5" (at 218.44 115.57 0)
+    (effects (font (size 1.27 1.27)) (justify left bottom))
+  )
+  (text "Joystick A0-A2" (at 219.71 157.48 0)
+    (effects (font (size 1.27 1.27)) (justify left bottom))
   )
   (global_label "A2" (shape input) (at 148.59 60.96 90) (fields_autoplaced)

Commit message: -
Other:
- note added: "Black"
- note added: "Col D7-D10 Row D2-D6"
- note added: "Red"
- note added: "White"
- note removed: "Col D7-D10 Row D2-D5"
Changed lines of the file:
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@@
     (stroke (width 0) (type default))
   )
-  (text "Col D7-D10 Row D2-D5" (at 218.44 115.57 0)
+  (text "Col D7-D10 Row D2-D6" (at 218.44 115.57 0)
     (effects (font (size 1.27 1.27)) (justify left bottom))
+  )
+  (text "White" (at 148.59 69.85 0)
+    (effects (font (size 1 1)) (justify left bottom))
+  )
+  (text "Red" (at 148.59 64.77 0)
+    (effects (font (size 1 1)) (justify left bottom))
   )
   (text "Joystick A0-A2" (at 219.71 157.48 0)
     (effects (font (size 1.27 1.27)) (justify left bottom))
   )
+  (text "Black" (at 148.59 67.31 0)
+    (effects (font (size 1 1)) (justify left bottom))
+  )
   (global_label "A2" (shape input) (at 148.59 60.96 90) (fields_autoplaced)
